File: PCB/mp3player/mp3player.kicad_sch (KiCad schematic)
At the start: 68 parts, among them J1 AudioJack3, J2 Battery, J3 USB_C, J4 Micro_SD_Card, J5 TFT SPI, SW1 Play, SW10 Power, SW2 Trk Prev, SW3 Trk Next, SW4 Mode Prev, SW5 Mode Next, SW6 Eq, SW7 Power, SW8 RESET, SW9 BOOT, U1 ESP32-S3-WROOM-1, U2 ES8388, U3 AP2112K-3.3, U4 MCP73831-2-OT, U5 USBLC6-2SC6

Commit message: added footprints
Parts:
- J1: footprint (none) -> Connector_Audio:Jack_3.5mm_CUI_SJ-3523-SMT_Horizontal
- J2: footprint (none) -> Connector_PinSocket_2.00mm:PinSocket_1x02_P2.00mm_Vertical
- J3: footprint (none) -> Connector_USB:USB_C_Receptacle_Amphenol_124019772112A
- J4: footprint (none) -> Connector_Card:microSD_HC_Wuerth_693072010801
- J5: footprint (none) -> Connector_PinSocket_2.00mm:PinSocket_1x08_P2.00mm_Vertical
- RV1: footprint (none) -> Potentiometer_SMD:Potentiometer_ACP_CA6-VSMD_Vertical
- SW1, SW10, SW2, SW3, SW4, SW5, SW6, SW7, SW9: footprint (none) -> Button_Switch_Keyboard:SW_Cherry_MX_1.00u_PCB
- SW8: footprint (none) -> Button_Switch_SMD:SW_Push_1P1T_NO_Vertical_Wuerth_434133025816
Changed lines of the file:
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@@
 			)
 		)
-		(property "Footprint" ""
+		(property "Footprint" "Button_Switch_Keyboard:SW_Cherry_MX_1.00u_PCB"
 			(at 60.96 110.49 0)
 			(hide yes)
@@
 			)
 		)
-		(property "Footprint" ""
+		(property "Footprint" "Button_Switch_Keyboard:SW_Cherry_MX_1.00u_PCB"
 			(at 181.61 133.35 0)
 			(hide yes)
@@
 			)
 		)
-		(property "Footprint" ""
+		(property "Footprint" "Button_Switch_Keyboard:SW_Cherry_MX_1.00u_PCB"
 			(at 43.18 142.24 0)
 			(hide yes)
@@
 			)
 		)
-		(property "Footprint" ""
+		(property "Footprint" "Connector_USB:USB_C_Receptacle_Amphenol_124019772112A"
 			(at 270.51 80.01 0)
 			(hide yes)
@@
 			)
 		)
-		(property "Footprint" ""
+		(property "Footprint" "Button_Switch_Keyboard:SW_Cherry_MX_1.00u_PCB"
 			(at 43.18 162.56 0)
 			(hide yes)
@@
 			)
 		)
-		(property "Footprint" ""
+		(property "Footprint" "Connector_PinSocket_2.00mm:PinSocket_1x02_P2.00mm_Vertical"
 			(at 292.1 27.94 0)
 			(hide yes)
@@
 			)
 		)
-		(property "Footprint" ""
+		(property "Footprint" "Connector_Card:microSD_HC_Wuerth_693072010801"
 			(at 162.56 184.15 0)
 			(hide yes)
@@
 			)
 		)
-		(property "Footprint" ""
+		(property "Footprint" "Button_Switch_Keyboard:SW_Cherry_MX_1.00u_PCB"
 			(at 43.18 152.4 0)
 			(hide yes)
@@
 			)
 		)
-		(property "Footprint" ""
+		(property "Footprint" "Potentiometer_SMD:Potentiometer_ACP_CA6-VSMD_Vertical"
 			(at 29.21 219.71 0)
 			(hide yes)
@@
 			)
 		)
-		(property "Footprint" ""
+		(property "Footprint" "Button_Switch_Keyboard:SW_Cherry_MX_1.00u_PCB"
 			(at 43.18 203.2 0)
 			(hide yes)
@@
 			)
 		)
-		(property "Footprint" ""
+		(property "Footprint" "Button_Switch_Keyboard:SW_Cherry_MX_1.00u_PCB"
 			(at 43.18 172.72 0)
 			(hide yes)
@@
 			)
 		)
-		(property "Footprint" ""
+		(property "Footprint" "Button_Switch_SMD:SW_Push_1P1T_NO_Vertical_Wuerth_434133025816"
 			(at 60.96 100.33 0)
 			(hide yes)
@@
 			)
 		)
-		(property "Footprint" ""
+		(property "Footprint" "Connector_PinSocket_2.00mm:PinSocket_1x08_P2.00mm_Vertical"
 			(at 232.41 139.7 0)
 			(hide yes)
@@
 			)
 		)
-		(property "Footprint" ""
+		(property "Footprint" "Connector_Audio:Jack_3.5mm_CUI_SJ-3523-SMT_Horizontal"
 			(at 203.2 53.34 0)
 			(hide yes)
@@
 			)
 		)
-		(property "Footprint" ""
+		(property "Footprint" "Button_Switch_Keyboard:SW_Cherry_MX_1.00u_PCB"
 			(at 43.18 182.88 0)
 			(hide yes)
@@
 			)
 		)
-		(property "Footprint" ""
+		(property "Footprint" "Button_Switch_Keyboard:SW_Cherry_MX_1.00u_PCB"
 			(at 43.18 193.04 0)
 			(hide yes)

Commit message: updated footprints, starting on pcb
Parts:
- added SW11: Next, Button_Switch_THT:SW_PUSH_6mm_H4.3mm, symbol Switch:SW_Push
- added SW12: Prev, Button_Switch_THT:SW_PUSH_6mm_H4.3mm, symbol Switch:SW_Push
- SW1, SW2, SW3, SW4, SW5, SW6, SW7, SW9: footprint Button_Switch_Keyboard:SW_Cherry_MX_1.00u_PCB -> Button_Switch_THT:SW_PUSH_6mm_H4.3mm
- SW10: value Power -> Power_sw; footprint Button_Switch_Keyboard:SW_Cherry_MX_1.00u_PCB -> Button_Switch_SMD:SW_DIP_SPSTx01_Slide_6.7x4.1mm_W6.73mm_P2.54mm_LowProfile_JPin
Connections:
- net GND: now also SW11.2, SW12.2
- net NEXT: now reaches U1.38 (IO2)
- net NEXT: now also SW11.1
- net PREV: now reaches U1.4 (IO4)
- net PREV: now also SW12.1
- no-connect marks 16 -> 14
Other:
- moved on the sheet: C16, RV1

Commit message: cont.
Parts:
- J5: footprint Connector_PinSocket_2.00mm:PinSocket_1x08_P2.00mm_Vertical -> Connector_JST:JST_GH_SM08B-GHS-TB_1x08-1MP_P1.25mm_Horizontal
Changed lines of the file:
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@@
 			)
 		)
-		(property "Footprint" "Connector_PinSocket_2.00mm:PinSocket_1x08_P2.00mm_Vertical"
+		(property "Footprint" "Connector_JST:JST_GH_SM08B-GHS-TB_1x08-1MP_P1.25mm_Horizontal"
 			(at 232.41 139.7 0)
 			(hide yes)

Commit message: worked on pcb
Parts:
- J2: footprint Connector_PinSocket_2.00mm:PinSocket_1x02_P2.00mm_Vertical -> Connector_PinSocket_2.00mm:PinSocket_1x02_P2.00mm_Horizontal
- SW8: footprint Button_Switch_SMD:SW_Push_1P1T_NO_Vertical_Wuerth_434133025816 -> Button_Switch_SMD:SW_SPST_PTS810
- SW9: footprint Button_Switch_THT:SW_PUSH_6mm_H4.3mm -> Button_Switch_SMD:SW_SPST_PTS810
Changed lines of the file:
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@@
 			)
 		)
-		(property "Footprint" "Button_Switch_THT:SW_PUSH_6mm_H4.3mm"
+		(property "Footprint" "Button_Switch_SMD:SW_SPST_PTS810"
 			(at 60.96 110.49 0)
 			(hide yes)
@@
 			)
 		)
-		(property "Footprint" "Connector_PinSocket_2.00mm:PinSocket_1x02_P2.00mm_Vertical"
+		(property "Footprint" "Connector_PinSocket_2.00mm:PinSocket_1x02_P2.00mm_Horizontal"
 			(at 292.1 27.94 0)
 			(hide yes)
@@
 			)
 		)
-		(property "Footprint" "Button_Switch_SMD:SW_Push_1P1T_NO_Vertical_Wuerth_434133025816"
+		(property "Footprint" "Button_Switch_SMD:SW_SPST_PTS810"
 			(at 60.96 100.33 0)
 			(hide yes)

Commit message: cont.
Connections:
- net CHG_PROG: now also U4.5 (PROG); no longer U4.1 (STAT)
- net CHG_STAT: now also U4.1 (STAT); no longer U4.5 (PROG)
- net VBAT: now also U4.3 (V_{BAT})
- no-connect marks 14 -> 13
Changed lines of the file:
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@@
-	)
-	(no_connect
-		(at 274.32 35.56)
 	)
 	(no_connect
@@
 		)
 	)
-	(label "CHG_PROG"
+	(label "CHG_STAT"
 		(at 274.32 40.64 270)
 		(effects
@@
 		)
 	)
+	(label "VBAT"
+		(at 274.32 35.56 0)
+		(effects
+			(font
+				(size 1.27 1.27)
+			)
+			(justify left bottom)
+		)
+	)
 	(label "IO0"
 		(at 21.59 40.64 0)
@@
 		)
 	)
-	(label "CHG_STAT"
+	(label "CHG_PROG"
 		(at 254 40.64 270)
 		(effects

Commit message: added BOM
Parts:
- R10, R11, R12, R13: value R -> 33
- R14, R15: value R -> 100k
Changed lines of the file:
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@@
 			)
 		)
-		(property "Value" "R"
+		(property "Value" "33"
 			(at 133.604 100.076 0)
 			(show_name no)
@@
 			)
 		)
-		(property "Value" "R"
+		(property "Value" "33"
 			(at 105.664 100.076 0)
 			(show_name no)
@@
 			)
 		)
-		(property "Value" "R"
+		(property "Value" "100k"
 			(at 106.68 139.6999 0)
 			(show_name no)
@@
 			)
 		)
-		(property "Value" "R"
+		(property "Value" "33"
 			(at 119.634 100.076 0)
 			(show_name no)
@@
 			)
 		)
-		(property "Value" "R"
+		(property "Value" "100k"
 			(at 106.68 147.3199 0)
 			(show_name no)
@@
 			)
 		)
-		(property "Value" "R"
+		(property "Value" "33"
 			(at 147.574 100.076 0)
 			(show_name no)
